Commit message: 地面归为

File: 6/src/fishbot_description/urdf/fishbot/base.urdf.xacro (robot description, xacro)
@@ -15,17 +15,4 @@
         </link>
     </xacro:macro>
-    <!-- ================= base_footprint 宏定义 =================
-         一个空的虚拟 link，用来表示"车体在地面上的投影"，
-         它才是整个机器人的 TF 根节点，base_link 位于它上方 height 处。
-         这样在 RViz 里把 Fixed Frame 选成 base_footprint，轮子就会刚好落在地面网格上。
-         height = 车体半高 + 轮子半径（本车 = 0.05 + 0.032 = 0.082）
-    -->
-    <xacro:macro name="base_footprint_xacro" params="height">
-        <link name="base_footprint"/>
-        <joint name="base_joint" type="fixed">
-            <parent link="base_footprint"/>
-            <child link="base_link"/>
-            <origin xyz="0 0 ${height}" rpy="0 0 0"/>
-        </joint>
-    </xacro:macro>
+    <!-- base_footprint（虚拟接地部件）已经独立到 base_footprint.urdf.xacro -->
 </robot>

File: 6/src/fishbot_description/urdf/fishbot/fishbot.urdf.xacro (robot description, xacro)
@@ -2,4 +2,5 @@
 <robot xmlns:xacro="http://www.ros.org/wiki/xacro" name="fishbot">
 <xacro:include filename="$(find fishbot_description)/urdf/fishbot/base.urdf.xacro"/>
+<xacro:include filename="$(find fishbot_description)/urdf/fishbot/base_footprint.urdf.xacro"/>
 <xacro:include filename="$(find fishbot_description)/urdf/fishbot/sensor/laser.urdf.xacro"/>
 <xacro:include filename="$(find fishbot_description)/urdf/fishbot/sensor/camera.urdf.xacro"/>
@@ -9,6 +10,7 @@
 <!-- 车体：半径 0.12、高 0.10 → 底面 z=-0.05，顶面 z=+0.05 -->
 <xacro:base_xacro radius="0.12" length="0.10"/>
-<!-- 虚拟接地参考系：base_link 在它上方 0.082
-     （0.082 = 车体半高 0.05 + 轮子半径 0.032，正好是轮底高度） -->
+<!-- 虚拟接地部件 base_footprint：车体在地面上的投影，也是整棵 TF 树的根
+     height = 车体半高 0.05 + 轮子半径 0.032 = 0.082 → 它的原点正好落在轮底（地面）上
+     RViz 里 Fixed Frame 选 base_footprint，四个轮子就会正好压在地面网格上 -->
 <xacro:base_footprint_xacro height="0.082"/>
 <!-- 传感器 -->
