Commit message: 6.5.2

File: 6/src/fishbot_description/urdf/fishbot/fishbot.urdf.xacro (robot description, xacro)
@@ -8,4 +8,7 @@
 <xacro:include filename="$(find fishbot_description)/urdf/actuator/wheel.urdf.xacro"/>
 <xacro:include filename="$(find fishbot_description)/urdf/actuator/caster.urdf.xacro"/>
+<!-- <xacro:include filename="$(find fishbot_description)/urdf/fishbot/plugins/gazebo_control_plugin.xacro"/> -->
+<xacro:include filename="$(find fishbot_description)/urdf/fishbot/plugins/gazebo_sensor_plugins.xacro"/>
+<xacro:include filename="$(find fishbot_description)/urdf/fishbot/fishbot.ros2_control.xacro" />
 <!-- 质量取值全部来自官方 chapt6 代码（ohhuo/ros2bookcode）：
      base 1.0 / imu 0.01 / 雷达杆 0.01 / 雷达 0.03 / 相机 0.01 / 驱动轮 0.1 / 支撑轮 0.01
@@ -36,3 +39,6 @@
 <xacro:caster_xacro name="front" xyz="0.08  0.0 -0.066" radius="0.016" mass="0.01"/>
 <xacro:caster_xacro name="rear"  xyz="-0.08 0.0 -0.066" radius="0.016" mass="0.01"/>
+<!-- <xacro:gazebo_control_plugin/> -->
+<xacro:gazebo_sensor_plugin/>
+<xacro:fishbot_ros2_control />
 </robot>

File: 6/src/fishbot_description/urdf/fishbot/sensor/camera.urdf.xacro (robot description, xacro)
@@ -24,4 +24,5 @@
             </collision>
         </link>
+        <link name="camera_optical_link"></link>
         <joint name="camera_joint" type="fixed">
             <parent link="base_link"/>
@@ -29,4 +30,9 @@
             <origin xyz="${xyz}" rpy="0 0 0"/>
         </joint>
+        <joint name="camera_optical_joint" type="fixed">
+            <parent link="camera_link"/>
+            <child link="camera_optical_link"/>
+            <origin xyz="0 0 0" rpy="${-pi/2} 0 ${-pi/2}"/>
+        </joint>
     </xacro:macro>
 </robot>

File: 6/src/fishbot_description/urdf/fishbot/sensor/laser.urdf.xacro (robot description, xacro)
@@ -55,4 +55,10 @@
             <origin xyz="${xyz}" rpy="0 0 0"/>
         </joint>
+        <gazebo reference="laser_cylinder_link">
+        <material>Gazebo/Black</material>
+        </gazebo>
+        <gazebo reference="laser_link">
+        <material>Gazebo/Black</material>
+        </gazebo>
     </xacro:macro>
 </robot>
