Commit message: 碰撞属性

File: 6/src/fishbot_description/urdf/actuator/caster.urdf.xacro (robot description, xacro)
@@ -17,4 +17,11 @@
                 </material>
             </visual>
+            <!-- collision 与 visual 保持同一套几何和 origin -->
+            <collision>
+                <origin xyz="0 0 0" rpy="0 0 0"/>
+                <geometry>
+                    <sphere radius="${radius}"/>
+                </geometry>
+            </collision>
         </link>
         <!-- 支撑轮只负责"撑住车身 + 被动跟随"，

File: 6/src/fishbot_description/urdf/actuator/wheel.urdf.xacro (robot description, xacro)
@@ -21,4 +21,12 @@
                 </material>
             </visual>
+            <!-- 碰撞体必须把 rpy="1.57079 0 0" 一起复制过来，
+                 否则碰撞圆柱会立着（轴向 Z），轮子在地面上会"陷进去" -->
+            <collision>
+                <origin xyz="0 0 0" rpy="1.57079 0 0"/>
+                <geometry>
+                    <cylinder radius="${radius}" length="${length}"/>
+                </geometry>
+            </collision>
         </link>
         <!-- 驱动轮要能一直转，所以用 continuous（而不是 revolute）

File: 6/src/fishbot_description/urdf/fishbot/base.urdf.xacro (robot description, xacro)
@@ -13,4 +13,13 @@
                 </material>
             </visual>
+            <!-- collision：碰撞属性，Gazebo 里真正参与物理计算的"硬外壳"
+                 这里和 visual 用同一套几何参数；为了省算力也可以简化成更粗的形状，
+                 但绝不能比 visual 大，否则机器人会看起来"悬空" -->
+            <collision>
+                <origin xyz="0 0 0" rpy="0 0 0"/>
+                <geometry>
+                    <cylinder radius="${radius}" length="${length}"/>
+                </geometry>
+            </collision>
         </link>
     </xacro:macro>

File: 6/src/fishbot_description/urdf/fishbot/sensor/camera.urdf.xacro (robot description, xacro)
@@ -14,4 +14,11 @@
                 </material>
             </visual>
+            <!-- collision 与 visual 保持同一套几何和 origin -->
+            <collision>
+                <origin xyz="0 0 0" rpy="0 0 0"/>
+                <geometry>
+                    <box size="0.02 0.10 0.02"/>
+                </geometry>
+            </collision>
         </link>
         <joint name="camera_joint" type="fixed">

File: 6/src/fishbot_description/urdf/fishbot/sensor/imu.urdf.xacro (robot description, xacro)
@@ -14,4 +14,11 @@
                 </material>
             </visual>
+            <!-- collision 与 visual 保持同一套几何和 origin -->
+            <collision>
+                <origin xyz="0 0 0" rpy="0 0 0"/>
+                <geometry>
+                    <box size="0.02 0.02 0.02"/>
+                </geometry>
+            </collision>
         </link>
         <joint name="imu_joint" type="fixed">

File: 6/src/fishbot_description/urdf/fishbot/sensor/laser.urdf.xacro (robot description, xacro)
@@ -14,4 +14,11 @@
                 </material>
             </visual>
+            <!-- 雷达支杆的碰撞体 -->
+            <collision>
+                <origin xyz="0 0 0" rpy="0 0 0"/>
+                <geometry>
+                     <cylinder radius="0.01" length="0.10"/>
+                </geometry>
+            </collision>
         </link>
         <link name="laser_link">
@@ -27,4 +34,11 @@
                 </material>
             </visual>
+            <!-- 雷达本体的碰撞体 -->
+            <collision>
+                <origin xyz="0 0 0" rpy="0 0 0"/>
+                <geometry>
+                     <cylinder radius="0.02" length="0.02"/>
+                </geometry>
+            </collision>
         </link>
         <joint name="laser_joint" type="fixed">

Commit message: 质量添加，惯性添加

File: 6/src/fishbot_description/urdf/actuator/caster.urdf.xacro (robot description, xacro)
@@ -1,4 +1,5 @@
 <?xml version="1.0"?>
 <robot xmlns:xacro="http://www.ros.org/wiki/xacro">
+    <xacro:include filename="$(find fishbot_description)/urdf/fishbot/common_inertia.xacro"/>
     <!-- ================= 万向支撑轮 宏定义 =================
          name   : front / rear，用来拼出 front_caster_link / front_caster_joint
@@ -6,6 +7,7 @@
          radius : 小球半径，取值要让"球底"和驱动轮轮底落在同一水平面
     -->
-    <xacro:macro name="caster_xacro" params="name xyz radius">
+    <xacro:macro name="caster_xacro" params="name xyz radius mass">
         <link name="${name}_caster_link">
+            <xacro:sphere_inertia m="${mass}" r="${radius}"/>
             <visual>
                 <origin xyz="0 0 0" rpy="0 0 0"/>
@@ -25,4 +27,15 @@
             </collision>
         </link>
+        <!-- 万向轮的摩擦配置（教程 6.3.2 的 1.3 小节）：
+             支撑轮是 fixed 固定死的、转不了，所以把摩擦系数设成 0，
+             让它在仿真里直接在地面上滑动，而不是"卡"住并且跟驱动轮抢地面。
+             mu1/mu2 是摩擦系数，kp/kd 是接触刚性/阻尼系数。
+             注意要放在 <link> 外面，<gazebo reference="..."> 是顶层标签。 -->
+        <gazebo reference="${name}_caster_link">
+            <mu1 value="0.0"/>
+            <mu2 value="0.0"/>
+            <kp value="1000000000.0"/>
+            <kd value="1.0"/>
+        </gazebo>
         <!-- 支撑轮只负责"撑住车身 + 被动跟随"，
              在 URDF 里用 fixed 就够了（真要让它滚，得配 Gazebo 的摩擦/万向轮插件，

File: 6/src/fishbot_description/urdf/actuator/wheel.urdf.xacro (robot description, xacro)
@@ -1,4 +1,5 @@
 <?xml version="1.0"?>
 <robot xmlns:xacro="http://www.ros.org/wiki/xacro">
+    <xacro:include filename="$(find fishbot_description)/urdf/fishbot/common_inertia.xacro"/>
     <!-- ================= 差速驱动轮 宏定义 =================
          name   : left / right，用来拼出 left_wheel_link / left_wheel_joint
@@ -7,6 +8,10 @@
          length : 轮子宽度，沿 Y 轴方向
     -->
-    <xacro:macro name="wheel_xacro" params="name xyz radius length">
+    <xacro:macro name="wheel_xacro" params="name xyz radius length mass">
         <link name="${name}_wheel_link">
+            <!-- 惯性宏按"圆柱轴向为 Z"推导，而轮子被 rpy 转到了 Y 向，
+                 所以要把同样的旋转传给宏（教程里没写这一项）。
+                 漏掉的话 izz（绕轮轴的转动惯量）会落到 Z 轴上，仿真里轮子会发飘 -->
+            <xacro:cylinder_inertia m="${mass}" r="${radius}" h="${length}" rpy="1.57079 0 0"/>
             <visual>
                 <!-- 圆柱默认轴向是 Z，绕 X 轴转 90° 后轴向变成 Y，轮子才立得起来。
@@ -30,4 +35,13 @@
             </collision>
         </link>
+        <!-- 驱动轮的摩擦配置（官方 chapt6 取值）：摩擦给得很大，
+             保证轮子能"抓住"地面把车推走，而不是原地打滑。
+             mu1/mu2 摩擦系数，kp/kd 接触刚性/阻尼 -->
+        <gazebo reference="${name}_wheel_link">
+            <mu1 value="20.0"/>
+            <mu2 value="20.0"/>
+            <kp value="1000000000.0"/>
+            <kd value="1.0"/>
+        </gazebo>
         <!-- 驱动轮要能一直转，所以用 continuous（而不是 revolute）
              axis 写在 child link 坐标系里，且 joint 的 origin 没有旋转，

File: 6/src/fishbot_description/urdf/fishbot/base.urdf.xacro (robot description, xacro)
@@ -1,7 +1,10 @@
 <?xml version="1.0"?>
 <robot xmlns:xacro="http://www.ros.org/wiki/xacro">
+    <!-- 官方做法：每个部件文件自己 include 一次惯性宏，这样单个文件也能独立展开 -->
+    <xacro:include filename="$(find fishbot_description)/urdf/fishbot/common_inertia.xacro"/>
     <!-- ================= base_link 宏定义 ================= -->
-    <xacro:macro name="base_xacro" params="radius length">
+    <xacro:macro name="base_xacro" params="radius length mass">
         <link name="base_link">
+            <xacro:cylinder_inertia m="${mass}" r="${radius}" h="${length}"/>
             <visual>
                 <origin xyz="0 0 0" rpy="0 0 0"/>

File: 6/src/fishbot_description/urdf/fishbot/fishbot.urdf.xacro (robot description, xacro)
@@ -8,25 +8,31 @@
 <xacro:include filename="$(find fishbot_description)/urdf/actuator/wheel.urdf.xacro"/>
 <xacro:include filename="$(find fishbot_description)/urdf/actuator/caster.urdf.xacro"/>
-<!-- 车体：半径 0.12、高 0.10 → 底面 z=-0.05，顶面 z=+0.05 -->
-<xacro:base_xacro radius="0.12" length="0.10"/>
+<!-- 质量取值全部来自官方 chapt6 代码（ohhuo/ros2bookcode）：
+     base 1.0 / imu 0.01 / 雷达杆 0.01 / 雷达 0.03 / 相机 0.01 / 驱动轮 0.1 / 支撑轮 0.01
+     合计 1.28kg。
+     官方是把质量写死在各个部件文件里的（m="0.1"），这里改成了宏参数，
+     好处是调质量只动这一处，惯性张量会自动跟着重算 -->
+<!-- 车体：半径 0.12、高 0.10 → 底面 z=-0.05，顶面 z=+0.05；质量 1.0kg -->
+<xacro:base_xacro radius="0.12" length="0.10" mass="1.0"/>
 <!-- 虚拟接地部件 base_footprint：车体在地面上的投影，也是整棵 TF 树的根
      height = 车体半高 0.05 + 轮子半径 0.032 = 0.082 → 它的原点正好落在轮底（地面）上
-     RViz 里 Fixed Frame 选 base_footprint，四个轮子就会正好压在地面网格上 -->
+     RViz 里 Fixed Frame 选 base_footprint，四个轮子就会正好压在地面网格上
+     虚拟 link 不加 inertial（没有质量，也不参与物理计算） -->
 <xacro:base_footprint_xacro height="0.082"/>
 <!-- 传感器 -->
-<xacro:imu_xacro xyz="0 0 0.02"/>
-<xacro:laser_xacro xyz="0 0.0 0.1"/>
+<xacro:imu_xacro xyz="0 0 0.02" mass="0.01"/>
+<xacro:laser_xacro xyz="0 0.0 0.1" cylinder_mass="0.01" laser_mass="0.03"/>
 <!-- 相机盒子高 0.02，顶面 z=0.05，故 z=0.06 时底面正好贴合顶面；
      x=0.11 时盒子占 x∈[0.10,0.12]，外侧面与半径 0.12 的圆柱面齐平 -->
-<xacro:camera_xacro xyz="0.11 0.0 0.06"/>
-<!-- ============ 左右差速驱动轮：半径 0.032、宽 0.04 ============
+<xacro:camera_xacro xyz="0.11 0.0 0.06" mass="0.01"/>
+<!-- ============ 左右差速驱动轮：半径 0.032、宽 0.04、各 0.1kg ============
      轮底 z = -0.05 - 0.032 = -0.082  ← 这就是"地面"的高度
      y = ±(0.12 + 0.04/2) = ±0.14，轮子内侧面正好贴住半径 0.12 的车体侧面 -->
-<xacro:wheel_xacro name="left"  xyz="0.0  0.14 -0.05" radius="0.032" length="0.04"/>
-<xacro:wheel_xacro name="right" xyz="0.0 -0.14 -0.05" radius="0.032" length="0.04"/>
-<!-- ============ 前后万向支撑轮：小球半径 0.016 ============
+<xacro:wheel_xacro name="left"  xyz="0.0  0.14 -0.05" radius="0.032" length="0.04" mass="0.1"/>
+<xacro:wheel_xacro name="right" xyz="0.0 -0.14 -0.05" radius="0.032" length="0.04" mass="0.1"/>
+<!-- ============ 前后万向支撑轮：小球半径 0.016、各 0.01kg ============
      球心 z = -0.082 + 0.016 = -0.066，球底与轮底齐平（都在 z=-0.082）
      球顶 z = -0.05，恰好与车体底面（z=-0.05）相切，像顶在底盘下面的一颗钢珠 -->
-<xacro:caster_xacro name="front" xyz="0.08  0.0 -0.066" radius="0.016"/>
-<xacro:caster_xacro name="rear"  xyz="-0.08 0.0 -0.066" radius="0.016"/>
+<xacro:caster_xacro name="front" xyz="0.08  0.0 -0.066" radius="0.016" mass="0.01"/>
+<xacro:caster_xacro name="rear"  xyz="-0.08 0.0 -0.066" radius="0.016" mass="0.01"/>
 </robot>

File: 6/src/fishbot_description/urdf/fishbot/sensor/camera.urdf.xacro (robot description, xacro)
@@ -1,7 +1,9 @@
 <?xml version="1.0"?>
 <robot xmlns:xacro="http://www.ros.org/wiki/xacro">
+    <xacro:include filename="$(find fishbot_description)/urdf/fishbot/common_inertia.xacro"/>
     <!-- ================= camera_link 宏定义 ================= -->
-    <xacro:macro name="camera_xacro" params="xyz">
+    <xacro:macro name="camera_xacro" params="xyz mass">
         <link name="camera_link">
+            <xacro:box_inertia m="${mass}" w="0.02" h="0.10" d="0.02"/>
             <visual>
                 <!-- visual 的 origin 是相对本 link 坐标系，偏移只写在 joint 上，这里必须为 0 -->

File: 6/src/fishbot_description/urdf/fishbot/sensor/imu.urdf.xacro (robot description, xacro)
@@ -1,7 +1,9 @@
 <?xml version="1.0"?>
 <robot xmlns:xacro="http://www.ros.org/wiki/xacro">
+    <xacro:include filename="$(find fishbot_description)/urdf/fishbot/common_inertia.xacro"/>
     <!-- ================= imu_link 宏定义 ================= -->
-    <xacro:macro name="imu_xacro" params="xyz">
+    <xacro:macro name="imu_xacro" params="xyz mass">
         <link name="imu_link">
+            <xacro:box_inertia m="${mass}" w="0.02" h="0.02" d="0.02"/>
             <visual>
                 <!-- visual 的 origin 是相对本 link 坐标系，偏移只写在 joint 上，这里必须为 0 -->

File: 6/src/fishbot_description/urdf/fishbot/sensor/laser.urdf.xacro (robot description, xacro)
@@ -1,7 +1,9 @@
 <?xml version="1.0"?>
 <robot xmlns:xacro="http://www.ros.org/wiki/xacro">
+    <xacro:include filename="$(find fishbot_description)/urdf/fishbot/common_inertia.xacro"/>
     <!-- ================= laser_link 宏定义 ================= -->
-    <xacro:macro name="laser_xacro" params="xyz">
+    <xacro:macro name="laser_xacro" params="xyz cylinder_mass laser_mass">
         <link name="laser_cylinder_link">
+            <xacro:cylinder_inertia m="${cylinder_mass}" r="0.01" h="0.10"/>
             <visual>
                 <!-- visual 的 origin 是相对本 link 坐标系，偏移只写在 joint 上，这里必须为 0 -->
@@ -23,4 +25,5 @@
         </link>
         <link name="laser_link">
+            <xacro:cylinder_inertia m="${laser_mass}" r="0.02" h="0.02"/>
             <visual>
                 <!-- 同 laser_cylinder_link：本 link 的几何体就在自己的坐标系原点，
