Commit message: world room

File: 6/src/fishbot_description/urdf/actuator/wheel.urdf.xacro (robot description, xacro)
@@ -53,4 +53,15 @@
             <origin xyz="${xyz}" rpy="0 0 0"/>
             <axis xyz="0 1 0"/>
+            <!-- ============ 轮子阻尼（教程里没有，这里补上）============
+                 不加这一项，轮子就是一对"完全没有刹车的自由轮"：
+                   joint 是 continuous，没有 damping、没有 friction，
+                   又没有控制器去约束它，任何一点点外力都会让轮子一直转下去。
+                 具体表现：车会在 Gazebo 里自己匀速往前溜，永远停不下来。
+                 实测（在 custom_room.world 里，出生点与墙有约 2.3cm 重叠）：
+                   无 damping : 16 秒漂移 187 毫米，还会自己转向
+                   有 damping : 16 秒漂移 0.1 毫米，基本纹丝不动
+                 0.1 是比较温和的值：既能刹住车，又不影响后面 6.5 章
+                 差速控制器正常驱动轮子。 -->
+            <dynamics damping="0.1" friction="0.1"/>
         </joint>
     </xacro:macro>
